Commit message: Initial commit

File: src/donar_robot_description/urdf/donar_robot.xacro (robot description, xacro)
@@ -65,5 +65,5 @@
 </link>
 <joint name="${frame_prefix}lidar_joint" type="fixed">
-  <origin xyz="0.36 0 0.645" rpy="0 0 0"/>
+  <origin xyz="0 0 0.765" rpy="0 0 0"/>
   <parent link="${frame_prefix}base_link"/>
   <child link="${frame_prefix}lidar_link"/>

Commit message: Initial commit of ROS2 warehouse robot project

File: src/donar_robot_description/urdf/donar_robot.xacro (robot description, xacro)
@@ -72,5 +72,5 @@
 <link name="${frame_prefix}right_wheel_1">
   <inertial>
-    <origin xyz="0.0 -0.0375 0.0" rpy="0 0 0"/>
+    <origin xyz="0 0 0" rpy="0 0 0"/>
     <mass value="6.75"/>
     <inertia ixx="0.12360346875" iyy="0.2371831875" izz="0.12360346875" ixy="0.0" iyz="0.0" ixz="0.0"/>
@@ -84,5 +84,8 @@
   </visual>
   <collision>
-    <origin xyz="0 -0.0375 0" rpy="1.57079632679 0 0"/>
+    <!-- Keep the wheel collision centered on the axle. Offsetting it from the
+         joint axis makes Gazebo simulate a skewed contact patch, which shows
+         up as sideways sliding and unwanted turning. -->
+    <origin xyz="0 0 0" rpy="1.57079632679 0 0"/>
     <geometry>
       <cylinder radius="0.21" length="0.075"/>
@@ -91,6 +94,6 @@
 </link>
 <gazebo reference="${frame_prefix}right_wheel_1">
-  <mu1>1.0</mu1>
-  <mu2>1.0</mu2>
+  <mu1>1.8</mu1>
+  <mu2>1.8</mu2>
   <kp>1000000.0</kp>
   <kd>100.0</kd>
@@ -105,5 +108,5 @@
 <link name="${frame_prefix}left_wheel_1">
   <inertial>
-    <origin xyz="0.0 0.0375 0.0" rpy="0 0 0"/>
+    <origin xyz="0 0 0" rpy="0 0 0"/>
     <mass value="6.75"/>
     <inertia ixx="0.12360346875" iyy="0.2371831875" izz="0.12360346875" ixy="0.0" iyz="0.0" ixz="0.0"/>
@@ -117,5 +120,5 @@
   </visual>
   <collision>
-    <origin xyz="0 0.0375 0" rpy="1.57079632679 0 0"/>
+    <origin xyz="0 0 0" rpy="1.57079632679 0 0"/>
     <geometry>
       <cylinder radius="0.21" length="0.075"/>
@@ -124,6 +127,6 @@
 </link>
 <gazebo reference="${frame_prefix}left_wheel_1">
-  <mu1>1.0</mu1>
-  <mu2>1.0</mu2>
+  <mu1>1.8</mu1>
+  <mu2>1.8</mu2>
   <kp>1000000.0</kp>
   <kd>100.0</kd>
@@ -152,5 +155,5 @@
     <origin xyz="0 0 -0.075" rpy="0 0 0"/>
     <geometry>
-      <sphere radius="0.06"/>
+      <sphere radius="0.045"/>
     </geometry>
   </collision>
@@ -164,8 +167,8 @@
 <!-- Add Gazebo friction properties -->
 <gazebo reference="${frame_prefix}left_caster_wheel_1">
-  <!-- Keep the fixed caster spheres low-friction so turns stay possible,
-       but not completely frictionless, which causes sideways skating. -->
-  <mu1>0.02</mu1>
-  <mu2>0.02</mu2>
+  <!-- Keep the fixed caster spheres fairly low-friction so turns stay
+       possible, but not so low that the robot skates sideways under load. -->
+  <mu1>0.12</mu1>
+  <mu2>0.12</mu2>
   <kp>1000000.0</kp>
   <kd>100.0</kd>
@@ -188,5 +191,5 @@
     <origin xyz="0 0 -0.075" rpy="0 0 0"/>
     <geometry>
-      <sphere radius="0.06"/>
+      <sphere radius="0.045"/>
     </geometry>
   </collision>
@@ -200,6 +203,6 @@
 <gazebo reference="${frame_prefix}right_caster_wheel_1">
   <!-- Match the left caster contact model to reduce lateral drift. -->
-  <mu1>0.02</mu1>
-  <mu2>0.02</mu2>
+  <mu1>0.12</mu1>
+  <mu2>0.12</mu2>
   <kp>1000000.0</kp>
   <kd>100.0</kd>
@@ -250,12 +253,12 @@
     <wheel_separation>0.78</wheel_separation>
     <wheel_radius>0.21</wheel_radius>
-    <max_linear_acceleration>3.0</max_linear_acceleration>
-    <min_linear_acceleration>-3.0</min_linear_acceleration>
-    <max_angular_acceleration>12.0</max_angular_acceleration>
-    <min_angular_acceleration>-12.0</min_angular_acceleration>
-    <max_linear_velocity>2.0</max_linear_velocity>
-    <min_linear_velocity>-2.0</min_linear_velocity>
-    <max_angular_velocity>6.0</max_angular_velocity>
-    <min_angular_velocity>-6.0</min_angular_velocity>
+    <max_linear_acceleration>0.9</max_linear_acceleration>
+    <min_linear_acceleration>-0.9</min_linear_acceleration>
+    <max_angular_acceleration>0.9</max_angular_acceleration>
+    <min_angular_acceleration>-0.9</min_angular_acceleration>
+    <max_linear_velocity>0.5</max_linear_velocity>
+    <min_linear_velocity>-0.25</min_linear_velocity>
+    <max_angular_velocity>0.55</max_angular_velocity>
+    <min_angular_velocity>-0.55</min_angular_velocity>
     <topic>/${robot_name}/cmd_vel</topic>
     <odom_topic>/${robot_name}/odometry</odom_topic>

Commit message: Initial commit

File: src/donar_robot_description/urdf/donar_robot.xacro (robot description, xacro)
@@ -146,5 +146,8 @@
   </inertial>
   <visual>
-    <origin xyz="0 0 -0.015" rpy="0 0 0"/>
+    <!-- Keep a tiny visual-only floor clearance so the caster does not look
+         sunken into the warehouse pad while leaving the contact geometry
+         unchanged. -->
+    <origin xyz="0 0 -0.003" rpy="0 0 0"/>
     <geometry>
       <sphere radius="0.12"/>
@@ -182,5 +185,5 @@
   </inertial>
   <visual>
-    <origin xyz="0 0 -0.015" rpy="0 0 0"/>
+    <origin xyz="0 0 -0.003" rpy="0 0 0"/>
     <geometry>
       <sphere radius="0.12"/>
